File: KiCad/RGB_SCART_VGA_Breakout.kicad_sch (KiCad schematic)
At the start: 24 parts, among them J1 SCART-F, J11 SJ1-3535NG, J2 Mini-DIN-4, J3 DE15_Plug_HighDensity_Mountin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, J4 Conn_01x09, J5 Mounting, J6 Mounting, J7 Mounting, J8 Mounting

Commit message: Update README.md.
Other:
- note added: "For jungle ICs with 0.7Vpp RGB inputs (like TDA8366): R1, R2, R3: 0 Ohm, R6, R7, R8: 75 Ohm. For jungle ICs with 0.5Vpp RGB inputs (like TA1276AN): R1, R2, R3: 30 Ohm, R6, R7, R8: 75 Ohm. Attenuation / divider resistors R1, R2, R3 can be changed to 24 Ohm, and termination resistors R6, R7, R8 to 51 Ohm for “proper” 75 Ohm termination."
- note removed: "For jungle ICs with 0.7Vpp RGB inputs (like TDA8366): R1, R2, R3: 0 Ohm, R6, R7, R8: 75 Ohm. For jungle ICs with 0.5Vpp RGB inputs (like TA1276AN): R1, R2, R3: 32 Ohm, R6, R7, R8: 75 Ohm. Attenuation / divider resistors R1, R2, R3 can be changed to 24 Ohm, and termination resistors R6, R7, R8 to 51 Ohm for “proper” 75 Ohm termination."
Changed lines of the file:
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@@
 	(generator_version "10.0")
 	(paper "A4")
-	(text "For jungle ICs with 0.7Vpp RGB inputs (like TDA8366):\nR1, R2, R3: 0 Ohm,\nR6, R7, R8: 75 Ohm.\n\nFor jungle ICs with 0.5Vpp RGB inputs (like TA1276AN):\nR1, R2, R3: 32 Ohm,\nR6, R7, R8: 75 Ohm.\nAttenuation / divider resistors R1, R2, R3 can be changed to 24 Ohm, \nand termination resistors R6, R7, R8 to 51 Ohm\nfor “proper” 75 Ohm termination."
+	(text "For jungle ICs with 0.7Vpp RGB inputs (like TDA8366):\nR1, R2, R3: 0 Ohm,\nR6, R7, R8: 75 Ohm.\n\nFor jungle ICs with 0.5Vpp RGB inputs (like TA1276AN):\nR1, R2, R3: 30 Ohm,\nR6, R7, R8: 75 Ohm.\nAttenuation / divider resistors R1, R2, R3 can be changed to 24 Ohm, \nand termination resistors R6, R7, R8 to 51 Ohm\nfor “proper” 75 Ohm termination."
 		(exclude_from_sim no)
 		(at 111.506 32.004 0)
